File: SCD/MK1/keyboard_mk1.kicad_sch (KiCad schematic)
At the start: 254 parts, among them K10 KEYSW, K100 KEYSW, K107 KEYSW, K108 KEYSW, K11 KEYSW, K111 KEYSW, K112 KEYSW, K113 KEYSW, K114 KEYSW, K115 KEYSW, K116 KEYSW, K117 KEYSW, K118 KEYSW, K119 KEYSW, K12 KEYSW, K120 KEYSW, K13 KEYSW, K14 KEYSW, K15 KEYSW, K16 KEYSW, K17 KEYSW, K18 KEYSW, K19 KEYSW, K20 KEYSW, K21 KEYSW, K22 KEYSW, K23 KEYSW, K24 KEYSW, K25 KEYSW, K26 KEYSW, K27 KEYSW, K28 KEYSW, K29 KEYSW, K30 KEYSW, K31 KEYSW, K32 KEYSW, K33 KEYSW, K34 KEYSW, K35 KEYSW, K36 KEYSW, K37 KEYSW, K38 KEYSW, K39 KEYSW, K4 KEYSW, K40 KEYSW, K41 KEYSW, K42 KEYSW, K43 KEYSW, K44 KEYSW, K45 KEYSW, K47 KEYSW, K48 KEYSW, K49 KEYSW, K5 KEYSW, K50 KEYSW, K51 KEYSW, K52 KEYSW, K53 KEYSW, K54 KEYSW, K55 KEYSW, K56 KEYSW, K57 KEYSW, K58 KEYSW, K59 KEYSW, K6 KEYSW, K61 KEYSW, K62 KEYSW, K63 KEYSW, K64 KEYSW, K65 KEYSW, K66 KEYSW, K67 KEYSW, K69 KEYSW, K7 KEYSW, K70 KEYSW, K71 KEYSW, K72 KEYSW, K73 KEYSW, K74 KEYSW, K75 KEYSW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

Commit message: Flipped stabilizer direction and added some silkscreen
Parts:
- 225K101, 225K110: footprint MX_Alps_Hybrid:MXOnly-2.25U-Hotswap-ReversedStabilizers -> MX_Alps_Hybrid:MXOnly-2.25U-Hotswap
- 275K121: footprint MX_Alps_Hybrid:MXOnly-2.75U-Hotswap-ReversedStabilizers -> MX_Alps_Hybrid:MXOnly-2.75U-Hotswap
- 2K106, 2K46, 2K60, 2K88: footprint MX_Alps_Hybrid:MXOnly-2U-Hotswap-ReversedStabilizers -> MX_Alps_Hybrid:MXOnly-2U-Hotswap
- 625K109: footprint MX_Alps_Hybrid:MXOnly-6.25U-Hotswap-ReversedStabilizers -> MX_Alps_Hybrid:MXOnly-6.25U-Hotswap
Changed lines of the file:
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@@
       (effects (font (size 1.524 1.524)) hide)
     )
-    (property "Footprint" "MX_Alps_Hybrid:MXOnly-2U-Hotswap-ReversedStabilizers" (at 283.21 -80.01 0)
+    (property "Footprint" "MX_Alps_Hybrid:MXOnly-2U-Hotswap" (at 283.21 -80.01 0)
       (effects (font (size 1.524 1.524)) hide)
     )
@@
       (effects (font (size 1.524 1.524)) hide)
     )
-    (property "Footprint" "MX_Alps_Hybrid:MXOnly-2U-Hotswap-ReversedStabilizers" (at -11.43 -66.04 0)
+    (property "Footprint" "MX_Alps_Hybrid:MXOnly-2U-Hotswap" (at -11.43 -66.04 0)
       (effects (font (size 1.524 1.524)) hide)
     )
@@
       (effects (font (size 1.524 1.524)) hide)
     )
-    (property "Footprint" "MX_Alps_Hybrid:MXOnly-6.25U-Hotswap-ReversedStabilizers" (at 127 -26.67 0)
+    (property "Footprint" "MX_Alps_Hybrid:MXOnly-6.25U-Hotswap" (at 127 -26.67 0)
       (effects (font (size 1.524 1.524)) hide)
     )
@@
       (effects (font (size 1.524 1.524)) hide)
     )
-    (property "Footprint" "MX_Alps_Hybrid:MXOnly-2U-Hotswap-ReversedStabilizers" (at -62.23 -36.83 0)
+    (property "Footprint" "MX_Alps_Hybrid:MXOnly-2U-Hotswap" (at -62.23 -36.83 0)
       (effects (font (size 1.524 1.524)) hide)
     )
@@
       (effects (font (size 1.524 1.524)) hide)
     )
-    (property "Footprint" "MX_Alps_Hybrid:MXOnly-2U-Hotswap-ReversedStabilizers" (at -11.43 -43.18 0)
+    (property "Footprint" "MX_Alps_Hybrid:MXOnly-2U-Hotswap" (at -11.43 -43.18 0)
       (effects (font (size 1.524 1.524)) hide)
     )
@@
       (effects (font (size 1.524 1.524)) hide)
     )
-    (property "Footprint" "MX_Alps_Hybrid:MXOnly-2.75U-Hotswap-ReversedStabilizers" (at 261.62 -39.37 0)
+    (property "Footprint" "MX_Alps_Hybrid:MXOnly-2.75U-Hotswap" (at 261.62 -39.37 0)
       (effects (font (size 1.524 1.524)) hide)
     )
@@
       (effects (font (size 1.524 1.524)) hide)
     )
-    (property "Footprint" "MX_Alps_Hybrid:MXOnly-2.25U-Hotswap-ReversedStabilizers" (at 273.05 -54.61 0)
+    (property "Footprint" "MX_Alps_Hybrid:MXOnly-2.25U-Hotswap" (at 273.05 -54.61 0)
       (effects (font (size 1.524 1.524)) hide)
     )
@@
       (effects (font (size 1.524 1.524)) hide)
     )
-    (property "Footprint" "MX_Alps_Hybrid:MXOnly-2.25U-Hotswap-ReversedStabilizers" (at 21.59 -39.37 0)
+    (property "Footprint" "MX_Alps_Hybrid:MXOnly-2.25U-Hotswap" (at 21.59 -39.37 0)
       (effects (font (size 1.524 1.524)) hide)
     )

Commit message: Added debouncing and LED driving as well as a good name
Parts:
- added C1, C2: 0.01uF, Capacitor_SMD:C_0805_2012Metric_Pad1.18x1.45mm_HandSolder, symbol Device:C
- added Q1, Q2: Q_Dual_NMOS_S1G1D2S2G2D1, Package_TO_SOT_SMD:SOT-363_SC-70-6_Handsoldering, symbol Device:Q_Dual_NMOS_S1G1D2S2G2D1
- added R10, R11, R12, R6, R7, R8, R9: 10K, Resistor_SMD:R_0805_2012Metric_Pad1.20x1.40mm_HandSolder, symbol Device:R
- K1: renamed from 125K1; footprint MX_Alps_Hybrid:MXOnly-1.25U-Hotswap -> MX_Alps_Hybrid:MXOnly-1U-Hotswap
- K2: renamed from 125K2; footprint MX_Alps_Hybrid:MXOnly-1.25U-Hotswap -> MX_Alps_Hybrid:MXOnly-1U-Hotswap
- K3: renamed from 125K3; footprint MX_Alps_Hybrid:MXOnly-1.25U-Hotswap -> MX_Alps_Hybrid:MXOnly-1U-Hotswap
- R3, R4, R5: value 56 -> 120
Connections:
- net +5V: now also R3.2, R4.2, R5.2, U1.14 (5V); no longer D122.1 (K), D123.1 (K), D124.1 (K), SW1.C, U1.13 (GND), U2.12 (VSS), U2.2 (A1), U2.3 (A2), U3.12 (VSS), U3.21 (A0), U3.3 (A2)
- net ENC_A: now also C2.2, R9.2; no longer SW1.A
- net ENC_B: now also C1.2, R6.2; no longer SW1.B
- net LED1: now also Q1.2 (G), R10.1; no longer R5.2
- net LED2: now also Q1.5 (G), R11.1; no longer R4.2
- net LED3: now also Q2.2 (G), R12.1; no longer R3.2
- net VCC: now also R7.2, R8.2
- new net: R6.1, R7.1, SW1.B
- new net: D124.1 (K), Q1.6 (D)
- new net: R8.1, R9.1, SW1.A
- new net: D122.1 (K), Q2.6 (D)
- new net: D123.1 (K), Q1.3 (D)
- new net GND: C1.1, C2.1, Q1.1 (S), Q1.4 (S), Q2.1 (S), R10.2, R11.2, R12.2, SW1.C, U1.13 (GND), U2.12 (VSS), U2.2 (A1), U2.3 (A2), U3.12 (VSS), U3.21 (A0), U3.3 (A2)
- no-connect marks 14 -> 18
Other:
- moved on the sheet: D122, D123, D124, R3, R4, R5
